Commit message: Replace the simulated robot with the one the CAD says can be built
urdf/ was aluminium cylinders with plausible masses and effort= values
derived from geometry: a fine simulation that could not be made. It is
now generated from cad/ - 17 CubeMars AK-series actuators, every mass
and inertia from the solids, every torque limit off a datasheet.

11.13 kg -> 21.89 kg. The interface is byte-for-byte the same shape -
20 bodies, 18 joints, 17 actuators, 86 sensors, 5 sites - so
climbing_env.py, the controller and the RL task load against it
unchanged. Vertical reach, which set the rung spacing, measures 0.676 m
against v1's 0.671.

Three things had to be fixed before any of it ran:

  The hanging keyframe settled at the reference rung's MIDPOINT, y=0.30.
  Every lesson scene in rl/ is laid out about y=0 and its start rung
  reaches only a little past it, so the left hook hung 47 mm off the end
  of lesson 1.35's rung and the robot fell 70 mm. It settles at y=0 now,
  and holds to 0.14 mm over 5 s.

  rl/lessons.py widened the shoulders by matching whole joint and
  actuator LINES. Those lines gained armature and frictionloss when the
  actuators became real, so the match would have stopped silently. It
  rewrites the range attribute instead, and asserts it hit something.

  The keyframe drift budget in the lesson smoke test goes 5 -> 8 mm.
  The keyframe is settled on scene.xml, the lessons add the grip pad,
  and the two equilibria differ by a few mm of contact compliance -
  which scales with weight, and the weight doubled.

cad/tools/verify.py passes all seven sections against this model:
masses sum, every inertia tensor is physically possible, MuJoCo loads
it, the joints match the spec and the datasheets, the worst torque
margin is 1.44x peak, and no legal pose self-intersects. All 18 lesson
scenes regenerate and pass their smoke checks.

What does NOT work yet, and is left that way deliberately: the
classical controller. Phases 0-2 pass - keyframe stability, hold map,
estimator and Jacobians - so the model is sound. Phases 3-8 time out or
fall, because every gain and move parameter in controller/ was tuned at
11 kg. Retuning is its own piece of work. Every trained PPO policy is
also void; they learned on the old robot.

One measurement worth chasing first: on the heavier robot the BARE hook
no longer slides along its rung the way it did. PAD_FRICTION and a
good deal of the curriculum exist to work around that slide.

Co-Authored-By: Claude Opus 5 <noreply@anthropic.com>

File: urdf/climbing_robot.urdf (robot description, URDF)
Before this commit: robot bimanual_wall_climber, 19 links, 18 joints
Links:
- link base_link: mass 4.395172 -> 4.389528; geometry collision cylinder length=0.067000 radius=0.039500; collision mesh filename=meshes/base_link_col.stl scale=0.001 0.001 0.001
- link fore_arm_L: mass 0.186534 -> 0.997296; geometry collision cylinder length=0.067000 radius=0.039500; collision mesh filename=meshes/fore_arm_L_col.stl scale=0.001 0.001 0.001
- link fore_arm_R: mass 0.186534 -> 0.997296; geometry collision cylinder length=0.067000 radius=0.039500; collision mesh filename=meshes/fore_arm_R_col.stl scale=0.001 0.001 0.001
- link forearm_rot_L: mass 0.076010 -> 0.826012; geometry collision cylinder length=0.067000 radius=0.039500; collision mesh filename=meshes/forearm_rot_L_col.stl scale=0.001 0.001 0.001
- link forearm_rot_R: mass 0.076010 -> 0.826012; geometry collision cylinder length=0.067000 radius=0.039500; collision mesh filename=meshes/forearm_rot_R_col.stl scale=0.001 0.001 0.001
- link hook_L: mass 0.123530 -> 0.266566; geometry collision box size=0.012000 0.065000 0.110000; collision box size=0.040000 0.065000 0.012000
- link hook_R: mass 0.123530 -> 0.266566; geometry collision box size=0.012000 0.065000 0.110000; collision box size=0.040000 0.065000 0.012000
- link humerus_rot_L: mass 0.090412 -> 0.959729; geometry collision cylinder length=0.061900 radius=0.049000; collision mesh filename=meshes/humerus_rot_L_col.stl scale=0.001 0.001 0.001
- link humerus_rot_R: mass 0.090412 -> 0.959729; geometry collision cylinder length=0.061900 radius=0.049000; collision mesh filename=meshes/humerus_rot_R_col.stl scale=0.001 0.001 0.001
- link shoulder_L: mass 0.075543 -> 1.256664; geometry collision cylinder length=0.061900 radius=0.049000; collision mesh filename=meshes/shoulder_L_col.stl scale=0.001 0.001 0.001
- link shoulder_R: mass 0.075543 -> 1.256664; geometry collision cylinder length=0.061900 radius=0.049000; collision mesh filename=meshes/shoulder_R_col.stl scale=0.001 0.001 0.001
- link torso_upper: mass 4.037000 -> 3.188336; geometry collision cylinder length=0.061900 radius=0.049000; collision cylinder length=0.061900 radius=0.049000
- link upper_arm_L: mass 0.293489 -> 1.292555; geometry collision cylinder length=0.061900 radius=0.049000; collision mesh filename=meshes/upper_arm_L_col.stl scale=0.001 0.001 0.001
- link upper_arm_R: mass 0.293489 -> 1.292555; geometry collision cylinder length=0.061900 radius=0.049000; collision mesh filename=meshes/upper_arm_R_col.stl scale=0.001 0.001 0.001
- link waist_link: mass 0.848230 -> 0.136650; geometry collision mesh filename=meshes/waist_link_col.stl scale=0.001 0.001 0.001; visual mesh filename=meshes/waist_link.stl scale=0.001 0.001 0.001
- link wrist_L: mass 0.040045 -> 0.942401; geometry collision cylinder length=0.067000 radius=0.039500; collision mesh filename=meshes/wrist_L_col.stl scale=0.001 0.001 0.001
- link wrist_R: mass 0.040045 -> 0.942401; geometry collision cylinder length=0.067000 radius=0.039500; collision mesh filename=meshes/wrist_R_col.stl scale=0.001 0.001 0.001
- link wrist_dev_L: mass 0.040045 -> 0.545989; geometry collision cylinder length=0.054000 radius=0.027500; collision mesh filename=meshes/wrist_dev_L_col.stl scale=0.001 0.001 0.001
- link wrist_dev_R: mass 0.040045 -> 0.545989; geometry collision cylinder length=0.054000 radius=0.027500; collision mesh filename=meshes/wrist_dev_R_col.stl scale=0.001 0.001 0.001
Joints:
- joint elbow_L: limit lower=-2.094395 upper=0.000000 effort=39 velocity=3.0 -> lower=-1.919862 upper=0.000000 effort=120 velocity=7.8540
- joint elbow_R: limit lower=-2.094395 upper=0.000000 effort=39 velocity=3.0 -> lower=-1.919862 upper=0.000000 effort=120 velocity=7.8540
- joint finger_L: limit lower=-1.570796 upper=0.349066 effort=13 velocity=3.0 -> lower=-1.570796 upper=0.349066 effort=24 velocity=5.4454; origin xyz=-0.000000 -0.000000 -0.020000 rpy=0 0 0 -> xyz=0.000000 0.000000 -0.072000 rpy=0 0 0
- joint finger_R: limit lower=-1.570796 upper=0.349066 effort=13 velocity=3.0 -> lower=-1.570796 upper=0.349066 effort=24 velocity=5.4454; origin xyz=0.000000 0.000000 -0.020000 rpy=0 0 0 -> xyz=0.000000 0.000000 -0.072000 rpy=0 0 0
- joint forearm_L_roll: limit lower=-1.483530 upper=1.483530 effort=23 velocity=3.0 -> lower=-1.483530 upper=1.483530 effort=72 velocity=10.2625; origin xyz=0.000000 -0.000000 -0.145000 rpy=0 0 0 -> xyz=0.000000 0.000000 -0.145000 rpy=0 0 0
- joint forearm_R_roll: limit lower=-1.483530 upper=1.483530 effort=23 velocity=3.0 -> lower=-1.483530 upper=1.483530 effort=72 velocity=10.2625
- joint shoulder_L_abduction: limit lower=0.000000 upper=3.141593 effort=68 velocity=3.0 -> lower=0.000000 upper=3.141593 effort=120 velocity=7.8540; origin xyz=-0.000000 0.125000 0.165000 rpy=0 0 0 -> xyz=0.000000 0.125000 0.269000 rpy=0 0 0
- joint shoulder_L_flexion: limit lower=-3.141593 upper=1.047198 effort=68 velocity=3.0 -> lower=-2.967060 upper=1.047198 effort=120 velocity=7.8540; origin xyz=0.000000 0.030000 0.000000 rpy=0 0 0 -> xyz=0.000000 0.030000 -0.104000 rpy=0 0 0
- joint shoulder_L_rotation: limit lower=-1.221730 upper=1.570796 effort=46 velocity=3.0 -> lower=-1.221730 upper=1.570796 effort=120 velocity=7.8540; origin xyz=0.000000 -0.000000 -0.200000 rpy=0 0 0 -> xyz=0.000000 0.000000 -0.200000 rpy=0 0 0
- joint shoulder_R_abduction: limit lower=-3.141593 upper=0.000000 effort=68 velocity=3.0 -> lower=-3.141593 upper=0.000000 effort=120 velocity=7.8540; origin xyz=0.000000 -0.125000 0.165000 rpy=0 0 0 -> xyz=0.000000 -0.125000 0.269000 rpy=0 0 0
- joint shoulder_R_flexion: limit lower=-3.141593 upper=1.047198 effort=68 velocity=3.0 -> lower=-2.967060 upper=1.047198 effort=120 velocity=7.8540; origin xyz=0.000000 -0.030000 0.000000 rpy=0 0 0 -> xyz=0.000000 -0.030000 -0.104000 rpy=0 0 0
- joint shoulder_R_rotation: limit lower=-1.570796 upper=1.221730 effort=46 velocity=3.0 -> lower=-1.570796 upper=1.221730 effort=120 velocity=7.8540
- joint waist_yaw: limit lower=-0.785398 upper=0.785398 effort=49 velocity=3.0 -> lower=-0.785398 upper=0.785398 effort=72 velocity=10.2625
- joint wrist_L_deviation: limit lower=-0.523599 upper=0.349066 effort=15 velocity=3.0 -> lower=-0.523599 upper=0.349066 effort=72 velocity=10.2625; origin xyz=0.000000 -0.000000 -0.020000 rpy=0 0 0 -> xyz=0.000000 0.000000 -0.084000 rpy=0 0 0
- joint wrist_L_flexion: limit lower=-0.436332 upper=0.436332 effort=17 velocity=3.0 -> lower=-0.436332 upper=0.436332 effort=72 velocity=10.2625
- joint wrist_R_deviation: limit lower=-0.349066 upper=0.523599 effort=15 velocity=3.0 -> lower=-0.349066 upper=0.523599 effort=72 velocity=10.2625; origin xyz=0.000000 -0.000000 -0.020000 rpy=0 0 0 -> xyz=0.000000 0.000000 -0.084000 rpy=0 0 0
- joint wrist_R_flexion: limit lower=-0.436332 upper=0.436332 effort=17 velocity=3.0 -> lower=-0.436332 upper=0.436332 effort=72 velocity=10.2625

File: urdf/climbing_robot_floating.urdf (robot description, URDF)
Before this commit: robot bimanual_wall_climber_floating, 20 links, 19 joints
Links:
- link base_link: mass 4.395172 -> 4.389528; geometry collision cylinder length=0.067000 radius=0.039500; collision mesh filename=meshes/base_link_col.stl scale=0.001 0.001 0.001
- link fore_arm_L: mass 0.186534 -> 0.997296; geometry collision cylinder length=0.067000 radius=0.039500; collision mesh filename=meshes/fore_arm_L_col.stl scale=0.001 0.001 0.001
- link fore_arm_R: mass 0.186534 -> 0.997296; geometry collision cylinder length=0.067000 radius=0.039500; collision mesh filename=meshes/fore_arm_R_col.stl scale=0.001 0.001 0.001
- link forearm_rot_L: mass 0.076010 -> 0.826012; geometry collision cylinder length=0.067000 radius=0.039500; collision mesh filename=meshes/forearm_rot_L_col.stl scale=0.001 0.001 0.001
- link forearm_rot_R: mass 0.076010 -> 0.826012; geometry collision cylinder length=0.067000 radius=0.039500; collision mesh filename=meshes/forearm_rot_R_col.stl scale=0.001 0.001 0.001
- link hook_L: mass 0.123530 -> 0.266566; geometry collision box size=0.012000 0.065000 0.110000; collision box size=0.040000 0.065000 0.012000
- link hook_R: mass 0.123530 -> 0.266566; geometry collision box size=0.012000 0.065000 0.110000; collision box size=0.040000 0.065000 0.012000
- link humerus_rot_L: mass 0.090412 -> 0.959729; geometry collision cylinder length=0.061900 radius=0.049000; collision mesh filename=meshes/humerus_rot_L_col.stl scale=0.001 0.001 0.001
- link humerus_rot_R: mass 0.090412 -> 0.959729; geometry collision cylinder length=0.061900 radius=0.049000; collision mesh filename=meshes/humerus_rot_R_col.stl scale=0.001 0.001 0.001
- link shoulder_L: mass 0.075543 -> 1.256664; geometry collision cylinder length=0.061900 radius=0.049000; collision mesh filename=meshes/shoulder_L_col.stl scale=0.001 0.001 0.001
- link shoulder_R: mass 0.075543 -> 1.256664; geometry collision cylinder length=0.061900 radius=0.049000; collision mesh filename=meshes/shoulder_R_col.stl scale=0.001 0.001 0.001
- link torso_upper: mass 4.037000 -> 3.188336; geometry collision cylinder length=0.061900 radius=0.049000; collision cylinder length=0.061900 radius=0.049000
- link upper_arm_L: mass 0.293489 -> 1.292555; geometry collision cylinder length=0.061900 radius=0.049000; collision mesh filename=meshes/upper_arm_L_col.stl scale=0.001 0.001 0.001
- link upper_arm_R: mass 0.293489 -> 1.292555; geometry collision cylinder length=0.061900 radius=0.049000; collision mesh filename=meshes/upper_arm_R_col.stl scale=0.001 0.001 0.001
- link waist_link: mass 0.848230 -> 0.136650; geometry collision mesh filename=meshes/waist_link_col.stl scale=0.001 0.001 0.001; visual mesh filename=meshes/waist_link.stl scale=0.001 0.001 0.001
- link wrist_L: mass 0.040045 -> 0.942401; geometry collision cylinder length=0.067000 radius=0.039500; collision mesh filename=meshes/wrist_L_col.stl scale=0.001 0.001 0.001
- link wrist_R: mass 0.040045 -> 0.942401; geometry collision cylinder length=0.067000 radius=0.039500; collision mesh filename=meshes/wrist_R_col.stl scale=0.001 0.001 0.001
- link wrist_dev_L: mass 0.040045 -> 0.545989; geometry collision cylinder length=0.054000 radius=0.027500; collision mesh filename=meshes/wrist_dev_L_col.stl scale=0.001 0.001 0.001
- link wrist_dev_R: mass 0.040045 -> 0.545989; geometry collision cylinder length=0.054000 radius=0.027500; collision mesh filename=meshes/wrist_dev_R_col.stl scale=0.001 0.001 0.001
Joints:
- joint elbow_L: limit lower=-2.094395 upper=0.000000 effort=39 velocity=3.0 -> lower=-1.919862 upper=0.000000 effort=120 velocity=7.8540
- joint elbow_R: limit lower=-2.094395 upper=0.000000 effort=39 velocity=3.0 -> lower=-1.919862 upper=0.000000 effort=120 velocity=7.8540
- joint finger_L: limit lower=-1.570796 upper=0.349066 effort=13 velocity=3.0 -> lower=-1.570796 upper=0.349066 effort=24 velocity=5.4454; origin xyz=-0.000000 -0.000000 -0.020000 rpy=0 0 0 -> xyz=0.000000 0.000000 -0.072000 rpy=0 0 0
- joint finger_R: limit lower=-1.570796 upper=0.349066 effort=13 velocity=3.0 -> lower=-1.570796 upper=0.349066 effort=24 velocity=5.4454; origin xyz=0.000000 0.000000 -0.020000 rpy=0 0 0 -> xyz=0.000000 0.000000 -0.072000 rpy=0 0 0
- joint forearm_L_roll: limit lower=-1.483530 upper=1.483530 effort=23 velocity=3.0 -> lower=-1.483530 upper=1.483530 effort=72 velocity=10.2625; origin xyz=0.000000 -0.000000 -0.145000 rpy=0 0 0 -> xyz=0.000000 0.000000 -0.145000 rpy=0 0 0
- joint forearm_R_roll: limit lower=-1.483530 upper=1.483530 effort=23 velocity=3.0 -> lower=-1.483530 upper=1.483530 effort=72 velocity=10.2625
- joint shoulder_L_abduction: limit lower=0.000000 upper=3.141593 effort=68 velocity=3.0 -> lower=0.000000 upper=3.141593 effort=120 velocity=7.8540; origin xyz=-0.000000 0.125000 0.165000 rpy=0 0 0 -> xyz=0.000000 0.125000 0.269000 rpy=0 0 0
- joint shoulder_L_flexion: limit lower=-3.141593 upper=1.047198 effort=68 velocity=3.0 -> lower=-2.967060 upper=1.047198 effort=120 velocity=7.8540; origin xyz=0.000000 0.030000 0.000000 rpy=0 0 0 -> xyz=0.000000 0.030000 -0.104000 rpy=0 0 0
- joint shoulder_L_rotation: limit lower=-1.221730 upper=1.570796 effort=46 velocity=3.0 -> lower=-1.221730 upper=1.570796 effort=120 velocity=7.8540; origin xyz=0.000000 -0.000000 -0.200000 rpy=0 0 0 -> xyz=0.000000 0.000000 -0.200000 rpy=0 0 0
- joint shoulder_R_abduction: limit lower=-3.141593 upper=0.000000 effort=68 velocity=3.0 -> lower=-3.141593 upper=0.000000 effort=120 velocity=7.8540; origin xyz=0.000000 -0.125000 0.165000 rpy=0 0 0 -> xyz=0.000000 -0.125000 0.269000 rpy=0 0 0
- joint shoulder_R_flexion: limit lower=-3.141593 upper=1.047198 effort=68 velocity=3.0 -> lower=-2.967060 upper=1.047198 effort=120 velocity=7.8540; origin xyz=0.000000 -0.030000 0.000000 rpy=0 0 0 -> xyz=0.000000 -0.030000 -0.104000 rpy=0 0 0
- joint shoulder_R_rotation: limit lower=-1.570796 upper=1.221730 effort=46 velocity=3.0 -> lower=-1.570796 upper=1.221730 effort=120 velocity=7.8540
- joint waist_yaw: limit lower=-0.785398 upper=0.785398 effort=49 velocity=3.0 -> lower=-0.785398 upper=0.785398 effort=72 velocity=10.2625
- joint wrist_L_deviation: limit lower=-0.523599 upper=0.349066 effort=15 velocity=3.0 -> lower=-0.523599 upper=0.349066 effort=72 velocity=10.2625; origin xyz=0.000000 -0.000000 -0.020000 rpy=0 0 0 -> xyz=0.000000 0.000000 -0.084000 rpy=0 0 0
- joint wrist_L_flexion: limit lower=-0.436332 upper=0.436332 effort=17 velocity=3.0 -> lower=-0.436332 upper=0.436332 effort=72 velocity=10.2625
- joint wrist_R_deviation: limit lower=-0.349066 upper=0.523599 effort=15 velocity=3.0 -> lower=-0.349066 upper=0.523599 effort=72 velocity=10.2625; origin xyz=0.000000 -0.000000 -0.020000 rpy=0 0 0 -> xyz=0.000000 0.000000 -0.084000 rpy=0 0 0
- joint wrist_R_flexion: limit lower=-0.436332 upper=0.436332 effort=17 velocity=3.0 -> lower=-0.436332 upper=0.436332 effort=72 velocity=10.2625
