Commit message: Audit the real-actuator robot: hooks the right way round, no phantom hulls, RL baselines read off the model
The robot swap loaded cleanly, and `python -m rl.climb_task` failed its own
incentive test: hanging still cost -58 over lesson 1 against -10 for a fall.
Four defects, each fixed where it comes from:

  Hooks back to front. dc2f07b's re-mount (the hook turned 180 deg about the
  forearm axis) lived only in the hand-edited scene.xml, and regenerating from
  cad/ dropped it: at the keyframe the throat faced away from the wall and both
  wrists leaned on it. It is spec.MOUNT_ROT now - fk, the URDF's finger joints,
  the scene's hook bodies - and the hook is drawn in its turned frame, so its
  plate stays on the flange side. The keyframe rolls the forearms -+5 as v1's
  did; -+5 of wrist flexion is not mirror-symmetric and hung 208 N on one hook
  and 100 N on the other. The hands start at y = +-0.155 again, where every
  lesson's goals and the controller's HANG expect them.

  Phantom self-collision. MuJoCo collides each mesh's hull, and one mesh per
  link made the torso frame one hull: the raised arms sank 10-22 mm into it,
  18-52 mm from any metal - 1500 N at the keyframe and four shoulder actuators
  at 88 % of peak. One collision mesh per CAD part now (stored as its hull),
  each wishbone arm split into ring and strip: of the self-contacts reported in
  the climbing envelope 14 % are hull artefacts, down from 71 %, and every real
  one is kept. The hang holds on <= 3.2 N.m a joint, and the sim runs 790
  control steps/s per process where it ran 440.

  Reward baselines typed for the 11 kg robot. TAU_IDLE 30 N.m and WEIGHT 109 N
  are ClimbTask.tau_idle (measured at the first reset, ~61) and .weight (from
  the model, 215). The self-checks' side pulls are fractions of body weight -
  friction holds a hook along its rung and scales with the load - and so are
  phase 7's; the SLAM wander bound is 30 mm for a 1.5x longer lever. A still
  hang now costs -7.81.

  1.5 GB per training env. MultiLesson compiles the lessons with discardvisual
  (bit-identical physics) over hull-only collision meshes: 0.33 GB per env.
  rl.render still loads the visuals.

Also: --resume refuses a checkpoint trained on another robot (state.json now
records a hash of scene.xml; --new-robot overrides), so none of the earlier,
now-void checkpoints can be continued by accident; phase 2 reads the IMU the
way the controller does, averaged over IMU_WINDOW, not one sample at the reset
instant; cad/src/robot.py imported a module that no longer exists; build123d's
.scale() ignores a part's Location (wrapped now); the lesson drift budget is
back at 5 mm (0.6 measured); stale README numbers.

Checked: rl.lessons 18/18, rl.climb_task OK, train_ppo --self-check OK,
cad/tools/verify.py 17/17, controller.test_climb phases 0-4 and 7 (5, 6 and 8
fall: their gains were tuned at 11 kg, deferred as before). PPO from scratch:
lesson -2 passed at 175k-950k steps depending on the seed, one run was still at
0 % after 1M; trained policies transfer between the collision models both ways.

Found, not fixed - a design call: at shoulder flexion -170 the upper arm's cheek
presses the wishbone ring by 1.4 mm, and trained policies hold -169.3 on 76-88 %
of their steps.

Co-Authored-By: Claude Opus 5 <noreply@anthropic.com>

File: urdf/climbing_robot.urdf (robot description, URDF)
Before this commit: robot bimanual_wall_climber_v2, 19 links, 18 joints
Links:
- link base_link: geometry collision cylinder length=0.067000 radius=0.039500; collision mesh filename=meshes/base_link_col_deck.stl scale=0.001 0.001 0.001
- link fore_arm_L: geometry collision cylinder length=0.067000 radius=0.039500; collision mesh filename=meshes/fore_arm_L_col_cheek.stl scale=0.001 0.001 0.001
- link fore_arm_R: geometry collision cylinder length=0.067000 radius=0.039500; collision mesh filename=meshes/fore_arm_R_col_cheek.stl scale=0.001 0.001 0.001
- link forearm_rot_L: geometry collision cylinder length=0.067000 radius=0.039500; collision mesh filename=meshes/forearm_rot_L_col_cheek.stl scale=0.001 0.001 0.001
- link forearm_rot_R: geometry collision cylinder length=0.067000 radius=0.039500; collision mesh filename=meshes/forearm_rot_R_col_cheek.stl scale=0.001 0.001 0.001
- link humerus_rot_L: geometry collision cylinder length=0.061900 radius=0.049000; collision mesh filename=meshes/humerus_rot_L_col_cheek.stl scale=0.001 0.001 0.001
- link humerus_rot_R: geometry collision cylinder length=0.061900 radius=0.049000; collision mesh filename=meshes/humerus_rot_R_col_cheek.stl scale=0.001 0.001 0.001
- link shoulder_L: geometry collision cylinder length=0.061900 radius=0.049000; collision mesh filename=meshes/shoulder_L_col_plate_face.stl scale=0.001 0.001 0.001
- link shoulder_R: geometry collision cylinder length=0.061900 radius=0.049000; collision mesh filename=meshes/shoulder_R_col_plate_face.stl scale=0.001 0.001 0.001
- link torso_upper: geometry collision cylinder length=0.061900 radius=0.049000; collision cylinder length=0.061900 radius=0.049000
- link upper_arm_L: geometry collision cylinder length=0.061900 radius=0.049000; collision mesh filename=meshes/upper_arm_L_col_cheek.stl scale=0.001 0.001 0.001
- link upper_arm_R: geometry collision cylinder length=0.061900 radius=0.049000; collision mesh filename=meshes/upper_arm_R_col_cheek.stl scale=0.001 0.001 0.001
- link waist_link: geometry collision mesh filename=meshes/waist_link_col_cone.stl scale=0.001 0.001 0.001; collision mesh filename=meshes/waist_link_col_flange.stl scale=0.001 0.001 0.001
- link wrist_L: geometry collision cylinder length=0.067000 radius=0.039500; collision mesh filename=meshes/wrist_L_col_plate_face.stl scale=0.001 0.001 0.001
- link wrist_R: geometry collision cylinder length=0.067000 radius=0.039500; collision mesh filename=meshes/wrist_R_col_plate_face.stl scale=0.001 0.001 0.001
- link wrist_dev_L: geometry collision cylinder length=0.054000 radius=0.027500; collision mesh filename=meshes/wrist_dev_L_col_plate_face.stl scale=0.001 0.001 0.001
- link wrist_dev_R: geometry collision cylinder length=0.054000 radius=0.027500; collision mesh filename=meshes/wrist_dev_R_col_plate_face.stl scale=0.001 0.001 0.001
Joints:
- joint finger_L: origin xyz=0.000000 0.000000 -0.072000 rpy=0 0 0 -> xyz=0.000000 0.000000 -0.072000 rpy=0 0 3.14159265
- joint finger_R: origin xyz=0.000000 0.000000 -0.072000 rpy=0 0 0 -> xyz=0.000000 0.000000 -0.072000 rpy=0 0 3.14159265

File: urdf/climbing_robot_floating.urdf (robot description, URDF)
Before this commit: robot bimanual_wall_climber_v2, 20 links, 19 joints
Links:
- link base_link: geometry collision cylinder length=0.067000 radius=0.039500; collision mesh filename=meshes/base_link_col_deck.stl scale=0.001 0.001 0.001
- link fore_arm_L: geometry collision cylinder length=0.067000 radius=0.039500; collision mesh filename=meshes/fore_arm_L_col_cheek.stl scale=0.001 0.001 0.001
- link fore_arm_R: geometry collision cylinder length=0.067000 radius=0.039500; collision mesh filename=meshes/fore_arm_R_col_cheek.stl scale=0.001 0.001 0.001
- link forearm_rot_L: geometry collision cylinder length=0.067000 radius=0.039500; collision mesh filename=meshes/forearm_rot_L_col_cheek.stl scale=0.001 0.001 0.001
- link forearm_rot_R: geometry collision cylinder length=0.067000 radius=0.039500; collision mesh filename=meshes/forearm_rot_R_col_cheek.stl scale=0.001 0.001 0.001
- link humerus_rot_L: geometry collision cylinder length=0.061900 radius=0.049000; collision mesh filename=meshes/humerus_rot_L_col_cheek.stl scale=0.001 0.001 0.001
- link humerus_rot_R: geometry collision cylinder length=0.061900 radius=0.049000; collision mesh filename=meshes/humerus_rot_R_col_cheek.stl scale=0.001 0.001 0.001
- link shoulder_L: geometry collision cylinder length=0.061900 radius=0.049000; collision mesh filename=meshes/shoulder_L_col_plate_face.stl scale=0.001 0.001 0.001
- link shoulder_R: geometry collision cylinder length=0.061900 radius=0.049000; collision mesh filename=meshes/shoulder_R_col_plate_face.stl scale=0.001 0.001 0.001
- link torso_upper: geometry collision cylinder length=0.061900 radius=0.049000; collision cylinder length=0.061900 radius=0.049000
- link upper_arm_L: geometry collision cylinder length=0.061900 radius=0.049000; collision mesh filename=meshes/upper_arm_L_col_cheek.stl scale=0.001 0.001 0.001
- link upper_arm_R: geometry collision cylinder length=0.061900 radius=0.049000; collision mesh filename=meshes/upper_arm_R_col_cheek.stl scale=0.001 0.001 0.001
- link waist_link: geometry collision mesh filename=meshes/waist_link_col_cone.stl scale=0.001 0.001 0.001; collision mesh filename=meshes/waist_link_col_flange.stl scale=0.001 0.001 0.001
- link wrist_L: geometry collision cylinder length=0.067000 radius=0.039500; collision mesh filename=meshes/wrist_L_col_plate_face.stl scale=0.001 0.001 0.001
- link wrist_R: geometry collision cylinder length=0.067000 radius=0.039500; collision mesh filename=meshes/wrist_R_col_plate_face.stl scale=0.001 0.001 0.001
- link wrist_dev_L: geometry collision cylinder length=0.054000 radius=0.027500; collision mesh filename=meshes/wrist_dev_L_col_plate_face.stl scale=0.001 0.001 0.001
- link wrist_dev_R: geometry collision cylinder length=0.054000 radius=0.027500; collision mesh filename=meshes/wrist_dev_R_col_plate_face.stl scale=0.001 0.001 0.001
Joints:
- joint finger_L: origin xyz=0.000000 0.000000 -0.072000 rpy=0 0 0 -> xyz=0.000000 0.000000 -0.072000 rpy=0 0 3.14159265
- joint finger_R: origin xyz=0.000000 0.000000 -0.072000 rpy=0 0 0 -> xyz=0.000000 0.000000 -0.072000 rpy=0 0 3.14159265

Commit message: Rebuild the shoulder pitch-first, the way the humanoids do it
Raised to hang, the arm grew out of a pivot BELOW the abduction motor and
folded back up past it - "arm up, shoulder pointing down" in the video. The
abduction-first stack put flexion 104 mm under the abduction axis; flaring the
raised arm swung its root 105 mm inward into the torso. Ten of twelve published
humanoids (Unitree H1/H1-2/G1, Booster T1, Fourier N1, Adam Lite, BHL,
ToddlerBot, OP3, iCub, Apollo, TALOS - measured off their own URDF/MJCF) put
shoulder PITCH on the torso and ROLL 27-78 mm outboard at the same height.
This robot does now:

  torso_upper -> flexion   y +-0.085, z 0.165, body inboard in the chest
  shoulder    -> abduction y +-0.070 further out, same height
  => the arm's root is at v1's (+-0.155, z 0.405) again

The brackets that changed, each through check_one / check_pair / check_swing:
shoulder_L is an L (a 17.5 mm web on the pitch output past the roll actuator's
flank, a leg across its far flange); upper_arm_L hangs off the roll output with
its cheek across the arm; torso_upper is a box - its side walls are the pitch
actuators' front-face plates, a deck, front, back and lid close it - 1.04 kg
against 1.49 for the yoke. Abduction stops inward at -12 (the upper arm meets
the shoulder bracket from -15; the survey stops at -7 to -25). 0 clashes over
the 17 joint pairs and 11 named poses; true CAD clear to flexion -180.

Downstream:
  - from the hang, positive abduction on the left IS the outward flare, and
    scene.xml has all of it: rl/lessons.py no longer widens anything and
    scene_wide_shoulders.xml is gone
  - each arm's qpos/ctrl order is flexion, then abduction; controller JOINTS
    follows and Estimator asserts the model's order; every earlier checkpoint
    is void (the robot stamp refuses it)
  - vertical reach is 0.56 m (4 seeds x 100k of _reach.py), not 0.68: the old
    number came from abducting 180 flipping the 104 mm shoulder link over the
    top, a 208 mm shrug no shoulder has. Rung rows are 0.45 m apart
  - 21.52 kg; hang drifts 0.08 mm / 5 s, <= 3.7 N.m a joint; torque margin
    >= 1.53x (box), 1.66x (envelope); shoulder flexion's worst case 74 -> 35 N.m
  - hull artefacts 2 % of the self-contacts in the climbing envelope (was 14)

Checks: verify.py all pass; rl.lessons, rl.climb_task, train_ppo --self-check
pass. PPO canary, 1.5M steps: lesson -2 passed before 100k, -1 at ~456k, 0 at
57 %. controller.test_climb passes 0, 1, 2, 4, 7 and fails 3, 5, 6, 8: phase
3's step lands 22 mm from its hold relative to the anchor, but the bare anchor
hook slides ~150 mm along the rung meanwhile (67 before) - the slide phase 7
measures; 5, 6, 8 fell before this too.

Co-Authored-By: Claude Opus 5 <noreply@anthropic.com>

File: urdf/climbing_robot.urdf (robot description, URDF)
Before this commit: robot bimanual_wall_climber_v2, 19 links, 18 joints
Links:
- link shoulder_L: mass 1.256664 -> 1.293615; geometry collision cylinder length=0.061900 radius=0.049000; collision mesh filename=meshes/shoulder_L_col_leg.stl scale=0.001 0.001 0.001
- link shoulder_R: mass 1.256664 -> 1.293615; geometry collision cylinder length=0.061900 radius=0.049000; collision mesh filename=meshes/shoulder_R_col_leg.stl scale=0.001 0.001 0.001
- link torso_upper: mass 3.188336 -> 2.743139; geometry collision cylinder length=0.061900 radius=0.049000; collision cylinder length=0.061900 radius=0.049000
Joints:
- joint shoulder_L_abduction: child shoulder_L -> upper_arm_L; limit lower=0.000000 upper=3.141593 effort=120 velocity=7.8540 -> lower=-0.209440 upper=3.141593 effort=120 velocity=7.8540; origin xyz=0.000000 0.125000 0.269000 rpy=0 0 0 -> xyz=0.000000 0.070000 0.000000 rpy=0 0 0; parent torso_upper -> shoulder_L
- joint shoulder_L_flexion: child upper_arm_L -> shoulder_L; origin xyz=0.000000 0.030000 -0.104000 rpy=0 0 0 -> xyz=0.000000 0.085000 0.165000 rpy=0 0 0; parent shoulder_L -> torso_upper
- joint shoulder_R_abduction: child shoulder_R -> upper_arm_R; limit lower=-3.141593 upper=0.000000 effort=120 velocity=7.8540 -> lower=-3.141593 upper=0.209440 effort=120 velocity=7.8540; origin xyz=0.000000 -0.125000 0.269000 rpy=0 0 0 -> xyz=0.000000 -0.070000 0.000000 rpy=0 0 0; parent torso_upper -> shoulder_R
- joint shoulder_R_flexion: child upper_arm_R -> shoulder_R; origin xyz=0.000000 -0.030000 -0.104000 rpy=0 0 0 -> xyz=0.000000 -0.085000 0.165000 rpy=0 0 0; parent shoulder_R -> torso_upper

File: urdf/climbing_robot_floating.urdf (robot description, URDF)
Before this commit: robot bimanual_wall_climber_v2, 20 links, 19 joints
Links:
- link shoulder_L: mass 1.256664 -> 1.293615; geometry collision cylinder length=0.061900 radius=0.049000; collision mesh filename=meshes/shoulder_L_col_leg.stl scale=0.001 0.001 0.001
- link shoulder_R: mass 1.256664 -> 1.293615; geometry collision cylinder length=0.061900 radius=0.049000; collision mesh filename=meshes/shoulder_R_col_leg.stl scale=0.001 0.001 0.001
- link torso_upper: mass 3.188336 -> 2.743139; geometry collision cylinder length=0.061900 radius=0.049000; collision cylinder length=0.061900 radius=0.049000
Joints:
- joint shoulder_L_abduction: child shoulder_L -> upper_arm_L; limit lower=0.000000 upper=3.141593 effort=120 velocity=7.8540 -> lower=-0.209440 upper=3.141593 effort=120 velocity=7.8540; origin xyz=0.000000 0.125000 0.269000 rpy=0 0 0 -> xyz=0.000000 0.070000 0.000000 rpy=0 0 0; parent torso_upper -> shoulder_L
- joint shoulder_L_flexion: child upper_arm_L -> shoulder_L; origin xyz=0.000000 0.030000 -0.104000 rpy=0 0 0 -> xyz=0.000000 0.085000 0.165000 rpy=0 0 0; parent shoulder_L -> torso_upper
- joint shoulder_R_abduction: child shoulder_R -> upper_arm_R; limit lower=-3.141593 upper=0.000000 effort=120 velocity=7.8540 -> lower=-3.141593 upper=0.209440 effort=120 velocity=7.8540; origin xyz=0.000000 -0.125000 0.269000 rpy=0 0 0 -> xyz=0.000000 -0.070000 0.000000 rpy=0 0 0; parent torso_upper -> shoulder_R
- joint shoulder_R_flexion: child upper_arm_R -> shoulder_R; origin xyz=0.000000 -0.030000 -0.104000 rpy=0 0 0 -> xyz=0.000000 -0.085000 0.165000 rpy=0 0 0; parent shoulder_R -> torso_upper

Commit message: Four Livox Mid-360 on the upper torso and a tube cage round them; the simulated robot rebuilt from the CAD at 24.16 kg
Two lidars on a roof over the head, 45 deg toward the wall and 45 deg away. Two more are
sunk into the chest and the back, only their windows outside, since the chest is
11-113 mm from the wall while climbing. Each bolts to a pad on a >= 3 mm plate, which
is Livox's condition for shedding its 6.5 W.

A cage of 16 x 2 mm 6061 tube guards all four: a bent bar up each corner of the torso,
40 mm proud of the panels, jogging in to y +-50 mm past the raised upper arms, and a
ring over the head at z 0.345 m joining their tops. Ray-casting picked that height:
lower costs the head lidars 8 % of what is above the hands.

The simulated robot, regenerated by gen_urdf.py and _gen_scene.py:
- Each lidar is a 265 g block. The mounts and the cage are the CAD solids. The total is
  21.52 -> 24.16 kg and the COM rises 136 -> 166 mm.
- Collision: the cage is 16 capsules on its centre lines, and each lidar a box and a
  cylinder as its STEP measures. The head's roof is one hull. The hats inside the
  torso meet nothing.
- A site marks each lidar's optical origin, and an occ_* site per collision geom tells
  the lidar model (rl/lidar.py) what it cannot see through.
- The visual mesh draws each lidar as its envelope. Livox's STEP is 54k triangles a
  unit, and four took torso_upper.stl past MuJoCo's 200k.
- The MJX robot pairs the cage capsules with every rung slot and wall: 1143 -> 1271
  pairs. The lidars inside the cage are dropped there.
- The keyframe was re-settled: 116 + 116 N on the hooks against 237 N, drifting under
  0.01 mm per 5 s. The torque tables were re-measured: the elbow's box margin is
  1.53x -> 1.37x, still over verify.py's 1.3x.

Checked: cad/tools/verify.py, 17 of 17. The keyframe hangs on every lesson for both
robots (rl.lessons, rl.mjx_scene). rl.mjx_check physics is OK. rl.mjx_check model: the
cage meets the wall in 10.8 % of states on both robots at 11.3 N. Its two gait
thresholds trip on win17's gait, which is from the old robot, so they need a policy
trained on this one.

controller.test_climb fails phases 4, 5, 6 and 8. It already failed four (3, 5, 6, 8)
on the commit before this.

Co-Authored-By: Claude Opus 5.5 <noreply@anthropic.com>

File: urdf/climbing_robot.urdf (robot description, URDF)
Before this commit: robot bimanual_wall_climber_v2, 19 links, 18 joints
Links:
- link torso_upper: mass 2.743139 -> 5.390151; geometry collision box size=0.064800 0.064800 0.033000; collision box size=0.064800 0.064800 0.033000

File: urdf/climbing_robot_floating.urdf (robot description, URDF)
Before this commit: robot bimanual_wall_climber_v2, 20 links, 19 joints
Links:
- link torso_upper: mass 2.743139 -> 5.390151; geometry collision box size=0.064800 0.064800 0.033000; collision box size=0.064800 0.064800 0.033000
